File: PCB/HRS/HRS.kicad_sch (KiCad schematic)
At the start: 16 parts, among them J1 Breakout_Conn, J2 TFT_Conn, SW1 ET02_Power_Switch, U1 TME_1205S

Commit message: Made PCBs
Connections:
- net 3.3_V: now also J1.3 (Pin_3); no longer J1.15 (Pin_15)
- net 5V: now also U1.4 (5V); no longer U1. (GND_5V)
- net 5V_CTL: now also PCB2.23 (GPIO); no longer PCB2.21 (GPIO)
- net AGND: now also J1.4 (Pin_4), PCB2.AG (GND); no longer J1.1 (Pin_1), PCB2.G (GND)
- net CLR_DATA: now also J1.14 (Pin_14); no longer J1.12 (Pin_12)
- net CLR_PIX: now also J1.12 (Pin_12); no longer J1.10 (Pin_10)
- net CS: now also J1.8 (Pin_8); no longer J1.5 (Pin_5)
- net DATA_RDY: now also J1.13 (Pin_13); no longer J1.11 (Pin_11)
- net GND: now also BT1.2 (-), C2.1, J1.1 (Pin_1), LD1.2 (GND), PCB2.G (GND), U1.1 (GND_12V), U1.3 (GND_5V); no longer J1.2 (Pin_2), LD1. (Vin), PCB2. (GND), U1. (GND_5V)
- net MISO: now also J1.9 (Pin_9); no longer J1.7 (Pin_7)
- net PWR_DOWN: now also J1.15 (Pin_15); no longer J1.13 (Pin_13)
- net READ: now also J1.7 (Pin_7); no longer J1.8 (Pin_8)
- net SCL: now also J1.10 (Pin_10); no longer J1.6 (Pin_6)
- net SCLK: now also J1.5 (Pin_5); no longer J1.3 (Pin_3)
- net SDATA: now also J1.6 (Pin_6); no longer J1.4 (Pin_4)
- net SHUTTER: now also J1.11 (Pin_11); no longer J1.9 (Pin_9)
- net VDD_5V: now also J1.2 (Pin_2); no longer J1.14 (Pin_14)
- net Y_Pos: now also PCB2.21 (A7); no longer PCB2.23 (A9)
- net at R1.1: now also LD1.1 (Vin); no longer LD1. (Vin)
- net at C2.2, SW1.2 (B): now also U1.2 (12V); no longer U1. (GND_5V)
Changed lines of the file:
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@@
     (stroke (width 0) (type default) (color 0 0 0 0))
   )
+  (label "GND" (at 95.25 46.99 0)
+    (effects (font (size 1.27 1.27)) (justify left bottom))
+  )
   (label "Status_LED" (at 148.59 96.52 0)
     (effects (font (size 1.27 1.27)) (justify left bottom))
   )
-  (label "Y_Pos" (at 148.59 101.6 0)
+  (label "Y_Pos" (at 137.16 87.63 90)
     (effects (font (size 1.27 1.27)) (justify left bottom))
   )
@@
     (effects (font (size 1.27 1.27)) (justify right bottom))
   )
-  (label "VDD_5V" (at 92.71 107.95 0)
+  (label "VDD_5V" (at 92.71 138.43 0)
     (effects (font (size 1.27 1.27)) (justify left bottom))
   )
@@
     (effects (font (size 1.27 1.27)) (justify right bottom))
   )
-  (label "DATA_RDY" (at 92.71 115.57 0)
+  (label "DATA_RDY" (at 92.71 110.49 0)
     (effects (font (size 1.27 1.27)) (justify left bottom))
   )
@@
     (effects (font (size 1.27 1.27)) (justify left bottom))
   )
-  (label "3.3_V" (at 92.71 105.41 0)
+  (label "3.3_V" (at 92.71 135.89 0)
     (effects (font (size 1.27 1.27)) (justify left bottom))
   )
@@
     (effects (font (size 1.27 1.27)) (justify left bottom))
   )
-  (label "5V_CTL" (at 137.16 87.63 90)
+  (label "5V_CTL" (at 148.59 101.6 0)
     (effects (font (size 1.27 1.27)) (justify left bottom))
   )
@@
     (effects (font (size 1.27 1.27)) (justify right bottom))
   )
-  (label "MISO" (at 92.71 125.73 0)
+  (label "MISO" (at 92.71 120.65 0)
     (effects (font (size 1.27 1.27)) (justify left bottom))
   )
@@
     (effects (font (size 1.27 1.27)) (justify right bottom))
   )
-  (label "GND" (at 92.71 138.43 0)
+  (label "GND" (at 92.71 140.97 0)
     (effects (font (size 1.27 1.27)) (justify left bottom))
   )
@@
     (effects (font (size 1.27 1.27)) (justify right bottom))
   )
-  (label "READ" (at 92.71 123.19 0)
+  (label "READ" (at 92.71 125.73 0)
     (effects (font (size 1.27 1.27)) (justify left bottom))
   )
@@
     (effects (font (size 1.27 1.27)) (justify right bottom))
   )
-  (label "CLR_DATA" (at 92.71 113.03 0)
+  (label "CLR_DATA" (at 92.71 107.95 0)
     (effects (font (size 1.27 1.27)) (justify left bottom))
   )
@@
     (effects (font (size 1.27 1.27)) (justify right bottom))
   )
-  (label "SCLK" (at 92.71 135.89 0)
+  (label "SCLK" (at 92.71 130.81 0)
     (effects (font (size 1.27 1.27)) (justify left bottom))
   )
@@
     (effects (font (size 1.27 1.27)) (justify left bottom))
   )
-  (label "SHUTTER" (at 92.71 120.65 0)
+  (label "SHUTTER" (at 92.71 115.57 0)
     (effects (font (size 1.27 1.27)) (justify left bottom))
   )
@@
     (effects (font (size 1.27 1.27)) (justify right bottom))
   )
-  (label "GND" (at 142.24 87.63 90)
-    (effects (font (size 1.27 1.27)) (justify left bottom))
-  )
-  (label "PWR_DOWN" (at 92.71 110.49 0)
-    (effects (font (size 1.27 1.27)) (justify left bottom))
-  )
-  (label "SCL" (at 92.71 128.27 0)
+  (label "GND" (at 144.78 121.92 270)
+    (effects (font (size 1.27 1.27)) (justify right bottom))
+  )
+  (label "PWR_DOWN" (at 92.71 105.41 0)
+    (effects (font (size 1.27 1.27)) (justify left bottom))
+  )
+  (label "SCL" (at 92.71 118.11 0)
     (effects (font (size 1.27 1.27)) (justify left bottom))
   )
@@
     (effects (font (size 1.27 1.27)) (justify right bottom))
   )
-  (label "AGND" (at 144.78 121.92 270)
-    (effects (font (size 1.27 1.27)) (justify right bottom))
+  (label "AGND" (at 142.24 87.63 90)
+    (effects (font (size 1.27 1.27)) (justify left bottom))
   )
   (label "LD" (at 139.7 57.15 270)
     (effects (font (size 1.27 1.27)) (justify right bottom))
   )
-  (label "CLR_PIX" (at 92.71 118.11 0)
+  (label "CLR_PIX" (at 92.71 113.03 0)
     (effects (font (size 1.27 1.27)) (justify left bottom))
   )
@@
     (effects (font (size 1.27 1.27)) (justify left bottom))
   )
-  (label "SDATA" (at 92.71 133.35 0)
-    (effects (font (size 1.27 1.27)) (justify left bottom))
-  )
-  (label "AGND" (at 92.71 140.97 0)
+  (label "SDATA" (at 92.71 128.27 0)
+    (effects (font (size 1.27 1.27)) (justify left bottom))
+  )
+  (label "AGND" (at 92.71 133.35 0)
     (effects (font (size 1.27 1.27)) (justify left bottom))
   )
@@
     (effects (font (size 1.27 1.27)) (justify right bottom))
   )
-  (label "CS" (at 92.71 130.81 0)
+  (label "CS" (at 92.71 123.19 0)
     (effects (font (size 1.27 1.27)) (justify left bottom))
   )
@@
   (symbol (lib_id "HRS:1054_LD") (at 138.43 41.91 270) (unit 1)
     (in_bom yes) (on_board yes)
-    (property "Reference" "LD1" (id 0) (at 138.43 33.02 90))
-    (property "Value" "1054_LD" (id 1) (at 138.43 35.56 90))
-    (property "Footprint" "HRS:BAT&LD" (id 2) (at 139.7 41.91 0)
-      (effects (font (size 1.27 1.27)) hide)
-    )
-    (property "Datasheet" "" (id 3) (at 139.7 41.91 0)
-      (effects (font (size 1.27 1.27)) hide)
-    )
-    (pin "")
-    (pin "")
+    (property "Reference" "LD1" (id 0) (at 147.32 41.91 90))
+    (property "Value" "1054_LD" (id 1) (at 144.78 41.91 90))
+    (property "Footprint" "HRS:BAT&LD" (id 2) (at 138.43 43.18 0)
+      (effects (font (size 1.27 1.27)) hide)
+    )
+    (property "Datasheet" "" (id 3) (at 138.43 43.18 0)
+      (effects (font (size 1.27 1.27)) hide)
+    )
+    (pin "1")
+    (pin "2")
   )
   (symbol (lib_id "Device:C") (at 91.44 41.91 180) (unit 1)
@@
       (effects (font (size 1.27 1.27)) hide)
     )
-    (pin "")
-    (pin "")
-    (pin "")
-    (pin "")
+    (pin "1")
+    (pin "2")
+    (pin "3")
+    (pin "4")
   )
   (symbol (lib_id "Switch:SW_SPST") (at 81.28 36.83 0) (unit 1)
@@
       (effects (font (size 1.27 1.27)) hide)
     )
-    (pin "")
+    (pin "AG")
     (pin "0")
     (pin "1")
